File: MakeFiles/V2X_ACCY.sch (KiCad schematic (older format))
At the start: 18 parts, among them P16 USB_u, U16 USB2422, U17 ADXL345, X2 24MHz

Commit message: Rev2.1 produced
Built R2.0, included findings, minor tweaks to placment and BOM.
Parts:
- C34, C35: Mouse PN 81-GRM188R71C105KA2J -> 581-06036C105MAT2A
- C37: Mouse PN 581-12063C475KAT2A -> 81-GRM21BR71A475KA3K
- P16: Mouse PN 656-DX4R005JJ2R1800 -> 798-ZX62D-B-5PA830
- U17: Mouse PN 584-ADXL345BCCZ-R7 -> 584-ADXL345BCCZ
Changed lines of the file:
@@
 3V3
 $Comp
-L GND #PWR82
+L GND #PWR074
 U 1 1 55F890DF
 P 3450 2300
-F 0 "#PWR82" H 3450 2050 50  0001 C CNN
+F 0 "#PWR074" H 3450 2050 50  0001 C CNN
 F 1 "GND" V 3450 2100 50  0000 C CNN
 F 2 "" H 3450 2300 60  0000 C CNN
@@
 HUB_CLKN
 $Comp
-L GND #PWR86
+L GND #PWR075
 U 1 1 55F89454
 P 5950 3150
-F 0 "#PWR86" H 5950 2900 50  0001 C CNN
+F 0 "#PWR075" H 5950 2900 50  0001 C CNN
 F 1 "GND" V 5950 2950 50  0000 C CNN
 F 2 "" H 5950 3150 60  0000 C CNN
@@
 $EndComp
 $Comp
-L GND #PWR88
+L GND #PWR076
 U 1 1 55F8A8AD
 P 6250 1450
-F 0 "#PWR88" H 6250 1200 50  0001 C CNN
+F 0 "#PWR076" H 6250 1200 50  0001 C CNN
 F 1 "GND" V 6250 1250 50  0000 C CNN
 F 2 "" H 6250 1450 60  0000 C CNN
@@
 $EndComp
 $Comp
-L GND #PWR85
+L GND #PWR077
 U 1 1 55F8AB65
 P 5100 950
-F 0 "#PWR85" H 5100 700 50  0001 C CNN
+F 0 "#PWR077" H 5100 700 50  0001 C CNN
 F 1 "GND" V 5100 750 50  0000 C CNN
 F 2 "" H 5100 950 60  0000 C CNN
@@
 $EndComp
 $Comp
-L GND #PWR75
+L GND #PWR078
 U 1 1 55F8AFDA
 P 1250 2050
-F 0 "#PWR75" H 1250 1800 50  0001 C CNN
+F 0 "#PWR078" H 1250 1800 50  0001 C CNN
 F 1 "GND" V 1250 1850 50  0000 C CNN
 F 2 "" H 1250 2050 60  0000 C CNN
@@
 $EndComp
 $Comp
-L GND #PWR78
+L GND #PWR079
 U 1 1 55F8B30B
 P 1750 1250
-F 0 "#PWR78" H 1750 1000 50  0001 C CNN
+F 0 "#PWR079" H 1750 1000 50  0001 C CNN
 F 1 "GND" V 1750 1050 50  0000 C CNN
 F 2 "" H 1750 1250 60  0000 C CNN
@@
 F 2 "CustomParts:C_0603_SM" H 1638 2000 30  0001 C CNN
 F 3 "http://www.mouser.com/ds/2/447/UPY-GPHC_X7R_6.3V-to-50V_8-12304.pdf" H 1600 2150 60  0001 C CNN
-F 4 "81-GRM188R71C105KA2J" H 1600 2150 60  0001 C CNN "Mouse PN"
+F 4 "581-06036C105MAT2A" H 1600 2150 60  0001 C CNN "Mouse PN"
 	1    1600 2150
 	1    0    0    -1
 $EndComp
 $Comp
-L GND #PWR76
+L GND #PWR080
 U 1 1 55F8B452
 P 1600 2300
-F 0 "#PWR76" H 1600 2050 50  0001 C CNN
+F 0 "#PWR080" H 1600 2050 50  0001 C CNN
 F 1 "GND" V 1600 2100 50  0000 C CNN
 F 2 "" H 1600 2300 60  0000 C CNN
@@
 $EndComp
 $Comp
-L GND #PWR84
+L GND #PWR081
 U 1 1 55F8B6A0
 P 4800 1350
-F 0 "#PWR84" H 4800 1100 50  0001 C CNN
+F 0 "#PWR081" H 4800 1100 50  0001 C CNN
 F 1 "GND" V 4800 1150 50  0000 C CNN
 F 2 "" H 4800 1350 60  0000 C CNN
@@
 HUB_SDA
 $Comp
-L GND #PWR89
+L GND #PWR082
 U 1 1 55F9C2E3
 P 6250 1700
-F 0 "#PWR89" H 6250 1450 50  0001 C CNN
+F 0 "#PWR082" H 6250 1450 50  0001 C CNN
 F 1 "GND" V 6250 1500 50  0000 C CNN
 F 2 "" H 6250 1700 60  0000 C CNN
@@
 F 2 "CustomParts:C_0603_SM" H 1788 950 30  0001 C CNN
 F 3 "http://www.mouser.com/ds/2/447/UPY-GPHC_X7R_6.3V-to-50V_8-12304.pdf" H 1750 1100 60  0001 C CNN
-F 4 "81-GRM188R71C105KA2J" H 1750 1100 60  0001 C CNN "Mouse PN"
+F 4 "581-06036C105MAT2A" H 1750 1100 60  0001 C CNN "Mouse PN"
 	1    1750 1100
 	1    0    0    -1
@@
 $EndComp
 $Comp
-L GND #PWR83
+L GND #PWR083
 U 1 1 5627872B
 P 4200 3250
-F 0 "#PWR83" H 4200 3000 50  0001 C CNN
+F 0 "#PWR083" H 4200 3000 50  0001 C CNN
 F 1 "GND" V 4200 3050 50  0000 C CNN
 F 2 "" H 4200 3250 60  0000 C CNN
@@
 F 1 "USB_u" H 1300 3400 50  0000 C CNN
 F 2 "CustomParts:USB_Micro-B-DX4R005JJ2R1800" V 1250 3100 60  0001 C CNN
-F 3 "http://www.mouser.com/ds/2/206/MB-0187-2E_DX4-221395.pdf" H 1250 3100 60  0001 C CNN
-F 4 "656-DX4R005JJ2R1800" H 1300 3200 60  0001 C CNN "Mouse PN"
+F 3 "http://www.mouser.com/ds/2/185/ZX_catalog-939768.pdf" H 1250 3100 60  0001 C CNN
+F 4 "798-ZX62D-B-5PA830" H 1300 3200 60  0001 C CNN "Mouse PN"
 	1    1300 3200
 	0    -1   1    0
@@
 HUB_DP
 $Comp
-L GND #PWR74
+L GND #PWR084
 U 1 1 567BADB1
 P 1200 3600
-F 0 "#PWR74" H 1200 3350 50  0001 C CNN
+F 0 "#PWR084" H 1200 3350 50  0001 C CNN
 F 1 "GND" V 1200 3400 50  0000 C CNN
 F 2 "" H 1200 3600 60  0000 C CNN
@@
 $EndComp
 $Comp
-L GND #PWR77
+L GND #PWR085
 U 1 1 567BADB7
 P 1600 3400
-F 0 "#PWR77" H 1600 3150 50  0001 C CNN
+F 0 "#PWR085" H 1600 3150 50  0001 C CNN
 F 1 "GND" V 1600 3200 50  0000 C CNN
 F 2 "" H 1600 3400 60  0000 C CNN
@@
 3V3
 $Comp
-L GND #PWR87
+L GND #PWR086
 U 1 1 567BB69B
 P 6250 1200
-F 0 "#PWR87" H 6250 950 50  0001 C CNN
+F 0 "#PWR086" H 6250 950 50  0001 C CNN
 F 1 "GND" V 6250 1000 50  0000 C CNN
 F 2 "" H 6250 1200 60  0000 C CNN
@@
 F 2 "CustomParts:LGA-14_5x3mm" H 3850 7200 60  0001 C CNN
 F 3 "http://www.mouser.com/ds/2/609/ADXL345-246395.pdf" H 3850 7200 60  0001 C CNN
-F 4 "584-ADXL345BCCZ-R7" H 3850 7200 60  0001 C CNN "Mouse PN"
+F 4 "584-ADXL345BCCZ" H 3850 7200 60  0001 C CNN "Mouse PN"
 	1    3850 7200
 	1    0    0    -1
 $EndComp
 $Comp
-L GND #PWR81
+L GND #PWR087
 U 1 1 567BDB94
 P 3400 7300
-F 0 "#PWR81" H 3400 7050 50  0001 C CNN
+F 0 "#PWR087" H 3400 7050 50  0001 C CNN
 F 1 "GND" H 3400 7150 50  0000 C CNN
 F 2 "" H 3400 7300 60  0000 C CNN
@@
 Connection ~ 3400 7300
 $Comp
-L GND #PWR79
+L GND #PWR088
 U 1 1 567BDB9D
 P 2000 7100
-F 0 "#PWR79" H 2000 6850 50  0001 C CNN
+F 0 "#PWR088" H 2000 6850 50  0001 C CNN
 F 1 "GND" H 2000 6950 50  0000 C CNN
 F 2 "" H 2000 7100 60  0000 C CNN
@@
 F 2 "CustomParts:C_0805_SM" H 2938 6800 30  0001 C CNN
 F 3 "http://www.yuden.co.jp/productdata/catalog/en/mlcc_all_e.pdf" H 2900 6950 60  0001 C CNN
-F 4 "581-12063C475KAT2A" H 2900 6950 60  0001 C CNN "Mouse PN"
+F 4 "81-GRM21BR71A475KA3K" H 2900 6950 60  0001 C CNN "Mouse PN"
 	1    2900 6950
 	1    0    0    -1
@@
 	2900 6800 3400 6800
 $Comp
-L GND #PWR80
+L GND #PWR089
 U 1 1 567BDBB4
 P 2900 7100
-F 0 "#PWR80" H 2900 6850 50  0001 C CNN
+F 0 "#PWR089" H 2900 6850 50  0001 C CNN
 F 1 "GND" H 2900 6950 50  0000 C CNN
 F 2 "" H 2900 7100 60  0000 C CNN
