File: MakeFiles/V2X_CTRL.sch (KiCad schematic (older format))
At the start: 37 parts, among them CON1 AVR-PDI-6, P20 Jumper 1, P21 Jumper 2, P22 CONN_02X04, P23 Jumper 3, P24 Jumper 4, Q16 2N7000, Q17 2N7000, Q18 2N7000, Q19 2N7000, U14 ATXMEGA16A4U-A, U21 74LS126, U22 74HC595, U23 74HC595

Commit message: 53851 Import of V2X R2.0
capture from legacy repo
Parts:
- removed C68: 1U, Custom Parts:C_0603_SM, symbol C
- removed C69: 100N, Custom Parts:C_0603_SM, symbol C
- removed D18, D19: 4148, Custom Parts:Diode_0805_12_SM, symbol D
- removed P20: Jumper 1, Fiducials:Fiducial_1mm_Dia_2.54mm_Outer_CopperTop, symbol CONN_01X01
- removed P21: Jumper 2, Fiducials:Fiducial_1mm_Dia_2.54mm_Outer_CopperTop, symbol CONN_01X01
- removed P22: CONN_02X04, Pin_Headers:Pin_Header_Straight_2x04, symbol CONN_02X04
- removed P23: Jumper 3, Fiducials:Fiducial_1mm_Dia_2.54mm_Outer_CopperTop, symbol CONN_01X01
- removed P24: Jumper 4, Fiducials:Fiducial_1mm_Dia_2.54mm_Outer_CopperTop, symbol CONN_01X01
- removed Q17, Q18, Q19: 2N7000, Custom Parts:SOT-23-123, symbol Q_NMOS_SGD
- removed R63: 1K, Custom Parts:R_0603_sm, symbol R
- removed R92, R93, R96: 47K, Custom Parts:R_0603_sm, symbol R
- removed R94: 22, Custom Parts:R_0603_sm, symbol R
- removed U21: 74LS126, Housings_SOIC:SOIC-14_3.9x8.7mm_Pitch1.27mm, symbol 74LS126
- removed U23: 74HC595, Housings_SOIC:SOIC-16_3.9x9.9mm_Pitch1.27mm, symbol 74HC595
- added C52: 100N, CustomParts:C_0603_SM, symbol C
- C41: renamed from C59; footprint Custom Parts:C_0603_SM -> CustomParts:C_0603_SM
- C42: renamed from C60; footprint Custom Parts:C_0603_SM -> CustomParts:C_0603_SM
- C43: renamed from C61; footprint Custom Parts:C_0603_SM -> CustomParts:C_0603_SM
- C44: renamed from C62; footprint Custom Parts:C_0603_SM -> CustomParts:C_0603_SM
- C45: renamed from C63; footprint Custom Parts:C_0603_SM -> CustomParts:C_0603_SM
- C46: renamed from C64; footprint Custom Parts:C_0603_SM -> CustomParts:C_0603_SM
- D11: renamed from D20; footprint LEDs:LED-0805 -> CustomParts:0805_LED; Mouse PN 720-LSR976-NR-1 -> 710-150080GS75000
- D12: renamed from D16; footprint LEDs:LED-0805 -> CustomParts:0805_LED; Mouse PN 720-LSR976-NR-1 -> 710-150080BS75000
- D13: renamed from D17; footprint LEDs:LED-0805 -> CustomParts:0805_LED; Mouse PN 710-150080BS75000 -> 710-150080RS75000
- FB4: renamed from FB6; footprint Custom Parts:R_0603_sm -> CustomParts:R_0603_sm
- PDI1: renamed from CON1; footprint Pin_Headers:Pin_Header_Angled_2x03 -> Pin_Headers:Pin_Header_Straight_2x03; Mouse PN 571-5-146130-2 -> 855-M20-9980346
- Q15: renamed from Q16; footprint Custom Parts:SOT-23-123 -> CustomParts:SOT_23_123; symbol Q_NMOS_SGD -> Q_NMOS_GSD
- R61: renamed from R95; footprint Custom Parts:R_0603_sm -> CustomParts:R_0603_sm
- R63: renamed from R90; value 330 -> 220; footprint Custom Parts:R_0603_sm -> CustomParts:R_0603_sm; Mouse PN 71-CRCW0603-330-E3 -> 71-CRCW0603-220-E3
- R66: renamed from R91; footprint Custom Parts:R_0603_sm -> CustomParts:R_0603_sm
- R67: renamed from R87; footprint Custom Parts:R_0603_sm -> CustomParts:R_0603_sm
- U20: renamed from U14; value ATXMEGA16A4U-A -> ATXMEGA128A4U-AU
- renumbered U22 to U18
Connections:
- net labels added: 3V3, 4V1, GPS_EN, HUB_PWR_PRT1, SEQ_DM, SEQ_DP, SIM_RESET
- net labels removed: 3V3_A, 3V3_B_EN, 3V3_C_EN, 3V3_D_EN, 3V3_E, ACCEL_RXD, ACCEL_TXD, CAN_BUF_FTDI, CAN_BUF_SEQ, CAN_RXD_FTDI, CAN_RXD_SEQ, FTDI_DM, FTDI_DP, HUB_ENABLE, HUB_SCL, HUB_SDA, HUB_STATUS, HUB_SUSP, SEQ_CHGPUMP, SEQ_RXD, SEQ_RXD_DM, SEQ_TXD, SEQ_TXD_DP, SIM_PWR, SIM_RF_OFF, SIM_VBUS, USB_INT_DM, USB_INT_DP, ~FTDI_RESET, ~SIM_RESET
- wire segments 35 -> 25
Other:
- note added: "4V1/3V3 Power Supply Enable (SIM)\n5V0 Power Supply Enable (CAN + HOST)\n5V0 HOST Enable \nELM/STN /Sleep\nELM/STN /Reset\nSIM Module "Power On"\nSIM Module /Reset\nSIM "Wake up""
- note added: "BUTTON Input\nAccelerometer Interupt 2 input\nAccelerometer Interupt 1 input\nHUB Power State Status input\nSystem Hibernate Supply Enable\nSEQ LED 1 Output\nSEQ LED 2 Output\nSEQ LED 3 Output"
- note added: "\nHost Short Circuit, Input/A2D\n\n\n"
- note removed: "3V3 Power Supply Enable (SEQ)\nHUB/FTDI 3V3 Enable\nCAN 3V3 Enable\nAccel 3V3 Enable\n4V1 Power Supply Enable (SIM)\n5V0 Power Supply Enable (LEDs)\n5V0 HOST Enable \nGSM module wake up signal"
- note removed: "BUTTON Input\nLED Charge pump Output\nAccelerometer Interupt 2 input\nAccelerometer Interupt 1 input\nHUB Suspend state input\nHUB Power State Status input\nSEQ LED 1 Output\nSEQ LED 2 Output"
- note removed: "CAN RXD BUFFER"
- note removed: "CAN_RXD_SEQ and CAN_RXD_FTDI\nare mutually exclusive siganls, only 1\ncan be logig high at any time.\nAllows only routing 2 TX source to CAN RXD"
- note removed: "HUB /RESET\nELM/STN /Reset\nELM/STN /Sleep\nSIM Module "Power On"\nSIM Module /Reset\nSIM "Airplane Mode"\nSIM USB detect\nFTDI USB detect /RESET"
- note removed: "HUB Serial Config Data I2C/SMB\nHUB Serial Config Clock I2C/SMB\nSEQ RXD to FTDI: ACL Data UART\nSEQ TXD to FTDI: ACL Data UART"
- note removed: "JUMPERS = 1-3, 2-4, 5-7, 6-8\nFTDI is USB with FTDI to SEQ control channel open\n\nJUMPERS = 3-5, 4-6\nAtmel is USB and FTDI disabled"
- note removed: "LED Charge pump. \nToggle pin state \nat approx 100khz"
- note removed: "SEQ LED3 Output\nHost Short Circuit, Input/A2D\nCAN RXD BUFFER: SEQ to CAN \nCAN RXD BUFFER: FTDI to CAN"
- note removed: "USB/UART signal Routing\nIf SW allows, FTDI can be removed from the system"
- moved on the sheet: C41, C42, D11, D12, D13, PDI1, R61, R63, R66, R67

Commit message: added high accuracy 32K crystal for RTC
only schematic
Parts:
- added C53, C54: 9p, CustomParts:C_0603_SM, symbol C
- added X3: 32.768K, Custom Parts:C_1206_SM, symbol Crystal_Small
Connections:
- net GND: now also C53.1, C54.1
- net at U20.36 (PR0/XTAL2/TOSC2): now also C54.2, X3.2
- net at U20.37 (PR1/XTAL1/TOSC1): now also C53.2, X3.1
- no-connect marks 9 -> 7
Changed lines of the file:
@@
 	0    -1   -1   0
 $EndComp
-NoConn ~ 3350 2100
-NoConn ~ 3350 2200
 $Comp
 L R R63
@@
 Text GLabel 5150 2000 2    60   Input ~ 0
 SEQ_LED1
+$Comp
+L Crystal_Small X3
+U 1 1 56DA0FEF
+P 2150 2100
+F 0 "X3" H 2150 2200 50  0000 C CNN
+F 1 "32.768K" H 2150 2250 50  0000 C CNN
+F 2 "Custom Parts:C_1206_SM" H 2150 2100 60  0001 C CNN
+F 3 "http://www.mouser.com/ds/2/360/SC-32P_Leaflet_r_newest-541780.pdf" H 2150 2100 60  0001 C CNN
+F 4 "628-SC32P-125PF20PPM" H 2150 2100 60  0001 C CNN "Mouser"
+	1    2150 2100
+	1    0    0    -1
+$EndComp
+$Comp
+L C C53
+U 1 1 56DA13C3
+P 1850 1950
+F 0 "C53" H 1875 2050 50  0000 L CNN
+F 1 "9p" H 1875 1850 50  0000 L CNN
+F 2 "CustomParts:C_0603_SM" H 1888 1800 30  0001 C CNN
+F 3 "http://www.mouser.com/ds/2/400/lcc_commercial_general_en-837201.pdf" H 1850 1950 60  0001 C CNN
+F 4 "DNS" H 1850 1950 60  0001 C CNN "Mouser"
+F 5 "810-C1608C0G1H090C" H 1850 1950 60  0001 C CNN "Mouse PN"
+	1    1850 1950
+	-1   0    0    -1
+$EndComp
+$Comp
+L C C54
+U 1 1 56DA1977
+P 2450 1950
+F 0 "C54" H 2475 2050 50  0000 L CNN
+F 1 "9p" H 2475 1850 50  0000 L CNN
+F 2 "CustomParts:C_0603_SM" H 2488 1800 30  0001 C CNN
+F 3 "http://www.mouser.com/ds/2/400/lcc_commercial_general_en-837201.pdf" H 2450 1950 60  0001 C CNN
+F 4 "DNS" H 2450 1950 60  0001 C CNN "Mouser"
+F 5 "810-C1608C0G1H090C" H 2450 1950 60  0001 C CNN "Mouse PN"
+	1    2450 1950
+	-1   0    0    -1
+$EndComp
+Wire Wire Line
+	2250 2100 3350 2100
+Connection ~ 2450 2100
+Wire Wire Line
+	2050 2100 1850 2100
+Wire Wire Line
+	1850 2100 1850 2200
+Wire Wire Line
+	1850 2200 3350 2200
+$Comp
+L GND #PWR0102
+U 1 1 56DA1E3F
+P 2450 1800
+F 0 "#PWR0102" H 2450 1550 50  0001 C CNN
+F 1 "GND" H 2450 1650 50  0000 C CNN
+F 2 "" H 2450 1800 60  0000 C CNN
+F 3 "" H 2450 1800 60  0000 C CNN
+	1    2450 1800
+	-1   0    0    1
+$EndComp
+$Comp
+L GND #PWR0103
+U 1 1 56DA2162
+P 1850 1800
+F 0 "#PWR0103" H 1850 1550 50  0001 C CNN
+F 1 "GND" H 1850 1650 50  0000 C CNN
+F 2 "" H 1850 1800 60  0000 C CNN
+F 3 "" H 1850 1800 60  0000 C CNN
+	1    1850 1800
+	-1   0    0    1
+$EndComp
 $EndSCHEMATC

Commit message: Changes for documentation
Other:
- moved on the sheet: U18
Changed lines of the file:
@@
 LIBS:xilinx
 LIBS:Zilog
+LIBS:CUSTOM_KICAD_PART
 LIBS:V2X-cache
 EELAYER 25 0
@@
 Text GLabel 6650 4450 2    60   Input ~ 0
 ~SIM_PWR_ON
-Text GLabel 2500 5750 2    60   Input ~ 0
+Text GLabel 3000 7100 2    60   Input ~ 0
 SIM_RESET
 Text GLabel 3350 3400 0    60   Input ~ 0
@@
 Text GLabel 3350 3200 0    60   Input ~ 0
 GPS_EN
-Text GLabel 2500 5150 2    60   Input ~ 0
+Text GLabel 3000 6500 2    60   Input ~ 0
 4V1_EN
-Text GLabel 2500 5250 2    60   Input ~ 0
+Text GLabel 3000 6600 2    60   Input ~ 0
 5V0_EN
 Text GLabel 3350 3000 0    60   Input ~ 0
 SIM_TXD
-Text GLabel 2500 5450 2    60   Input ~ 0
+Text GLabel 3000 6800 2    60   Input ~ 0
 ~CAN_SLEEP
-Text GLabel 2500 5550 2    60   Input ~ 0
+Text GLabel 3000 6900 2    60   Input ~ 0
 ~CAN_RESET
 Text Notes 6050 3600 0    69   ~ 0
@@
 Text Notes 8700 3000 0    60   ~ 0
 PDI (a-wire) Programing port
-Text Notes 3100 5900 0    69   ~ 0
+Text Notes 3600 7250 0    69   ~ 0
 4V1/3V3 Power Supply Enable (SIM)\n5V0 Power Supply Enable (CAN + HOST)\n5V0 HOST Enable \nELM/STN /Sleep\nELM/STN /Reset\nSIM Module "Power On"\nSIM Module /Reset\nSIM "Wake up"
 Text Notes 9700 3250 0    69   ~ 0
@@
 L 74HC595 U18
 U 1 1 55FA3B36
-P 1800 5600
-F 0 "U18" H 1950 6200 70  0000 C CNN
-F 1 "74HC595" H 1800 5000 70  0000 C CNN
-F 2 "Housings_SOIC:SOIC-16_3.9x9.9mm_Pitch1.27mm" H 1800 5600 60  0001 C CNN
-F 3 "http://www.mouser.com/ds/2/302/74HC_HCT595_Q100-269352.pdf" H 1800 5600 60  0001 C CNN
-F 4 "771-74HC595D-Q100" H 1800 5600 60  0001 C CNN "Mouse PN"
-	1    1800 5600
-	1    0    0    -1
-$EndComp
-Text GLabel 2500 5350 2    60   Input ~ 0
+P 2300 6950
+F 0 "U18" H 2450 7550 70  0000 C CNN
+F 1 "74HC595" H 2300 6350 70  0000 C CNN
+F 2 "Housings_SOIC:SOIC-16_3.9x9.9mm_Pitch1.27mm" H 2300 6950 60  0001 C CNN
+F 3 "http://www.mouser.com/ds/2/302/74HC_HCT595_Q100-269352.pdf" H 2300 6950 60  0001 C CNN
+F 4 "771-74HC595D-Q100" H 2300 6950 60  0001 C CNN "Mouse PN"
+	1    2300 6950
+	1    0    0    -1
+$EndComp
+Text GLabel 3000 6700 2    60   Input ~ 0
 5V0_B_EN
 $Comp
 L GND #PWR092
 U 1 1 55FA434A
-P 1100 5750
-F 0 "#PWR092" H 1100 5500 50  0001 C CNN
-F 1 "GND" H 1100 5600 50  0000 C CNN
-F 2 "" H 1100 5750 60  0000 C CNN
-F 3 "" H 1100 5750 60  0000 C CNN
-	1    1100 5750
+P 1600 7100
+F 0 "#PWR092" H 1600 6850 50  0001 C CNN
+F 1 "GND" H 1600 6950 50  0000 C CNN
+F 2 "" H 1600 7100 60  0000 C CNN
+F 3 "" H 1600 7100 60  0000 C CNN
+	1    1600 7100
 	1    0    0    -1
 $EndComp
@@
 Text GLabel 6100 4850 0    60   Input ~ 0
 SIM_PWR_ON
-Text GLabel 2500 5650 2    60   Input ~ 0
+Text GLabel 3000 7000 2    60   Input ~ 0
 SIM_PWR_ON
 Connection ~ 6650 4650
@@
 Text GLabel 7050 4650 2    60   Input ~ 0
 3V3
-Text GLabel 1100 5150 0    60   Input ~ 0
+Text GLabel 1600 6500 0    60   Input ~ 0
 SEQ_MOSI
-Text GLabel 1100 5650 0    60   Input ~ 0
+Text GLabel 1600 7000 0    60   Input ~ 0
 SR_LATCH
-Text GLabel 1100 5450 0    60   Input ~ 0
+Text GLabel 1600 6800 0    60   Input ~ 0
 SR_CLEAR
-Text GLabel 1100 5350 0    60   Input ~ 0
+Text GLabel 1600 6700 0    60   Input ~ 0
 SEQ_SCK
 Wire Notes Line
@@
 Text GLabel 5150 3100 2    60   Input ~ 0
 CAN_RXD
-Text GLabel 2500 5850 2    60   Input ~ 0
+Text GLabel 3000 7200 2    60   Input ~ 0
 SIM_WAKE
 NoConn ~ 9450 3550
@@
 Text GLabel 10650 4900 1    60   Input ~ 0
 4V1
-NoConn ~ 2500 6050
+NoConn ~ 3000 7400
 NoConn ~ 5150 2350
 NoConn ~ 5150 2550

Commit message: Part numer updates
for error or out of stock
Parts:
- C46: Mouse PN 603-CC603KRX7R7BB105 -> 81-GRM188R71C105KA2J
- U20: Mouse PN 556-ATXMEGA16A4U-AU -> 556-ATXMEGA128A4U-AU
- X3: Mouser 628-SC32P-125PF20PPM -> 815-S07AIG-32.76891T
Changed lines of the file:
@@
 SEQ_LED2
 $Comp
-L GND #PWR090
+L GND #PWR93
 U 1 1 55F86E9C
 P 4100 3900
-F 0 "#PWR090" H 4100 3650 50  0001 C CNN
+F 0 "#PWR93" H 4100 3650 50  0001 C CNN
 F 1 "GND" H 4100 3750 50  0000 C CNN
 F 2 "" H 4100 3900 60  0000 C CNN
@@
 PDI
 $Comp
-L GND #PWR091
+L GND #PWR102
 U 1 1 55F86EF0
 P 10000 3650
-F 0 "#PWR091" H 10000 3400 50  0001 C CNN
+F 0 "#PWR102" H 10000 3400 50  0001 C CNN
 F 1 "GND" H 10000 3500 50  0000 C CNN
 F 2 "" H 10000 3650 60  0000 C CNN
@@
 5V0_B_EN
 $Comp
-L GND #PWR092
+L GND #PWR90
 U 1 1 55FA434A
 P 1600 7100
-F 0 "#PWR092" H 1600 6850 50  0001 C CNN
+F 0 "#PWR90" H 1600 6850 50  0001 C CNN
 F 1 "GND" H 1600 6950 50  0000 C CNN
 F 2 "" H 1600 7100 60  0000 C CNN
@@
 $EndComp
 $Comp
-L GND #PWR093
+L GND #PWR94
 U 1 1 55FE1020
 P 6400 5050
-F 0 "#PWR093" H 6400 4800 50  0001 C CNN
+F 0 "#PWR94" H 6400 4800 50  0001 C CNN
 F 1 "GND" H 6400 4900 50  0000 C CNN
 F 2 "" H 6400 5050 60  0000 C CNN
@@
 Connection ~ 10550 750
 $Comp
-L GND #PWR094
+L GND #PWR103
 U 1 1 56006FBB
 P 10550 1100
-F 0 "#PWR094" H 10550 850 50  0001 C CNN
+F 0 "#PWR103" H 10550 850 50  0001 C CNN
 F 1 "GND" H 10550 950 50  0000 C CNN
 F 2 "" H 10550 1100 60  0000 C CNN
@@
 Connection ~ 9000 750
 $Comp
-L GND #PWR095
+L GND #PWR97
 U 1 1 560285A0
 P 9000 1100
-F 0 "#PWR095" H 9000 850 50  0001 C CNN
+F 0 "#PWR97" H 9000 850 50  0001 C CNN
 F 1 "GND" H 9000 950 50  0000 C CNN
 F 2 "" H 9000 1100 60  0000 C CNN
@@
 $EndComp
 $Comp
-L GND #PWR096
+L GND #PWR99
 U 1 1 560285F6
 P 9300 1100
-F 0 "#PWR096" H 9300 850 50  0001 C CNN
+F 0 "#PWR99" H 9300 850 50  0001 C CNN
 F 1 "GND" H 9300 950 50  0000 C CNN
 F 2 "" H 9300 1100 60  0000 C CNN
@@
 $EndComp
 $Comp
-L GND #PWR097
+L GND #PWR101
 U 1 1 5602864C
 P 9600 1100
-F 0 "#PWR097" H 9600 850 50  0001 C CNN
+F 0 "#PWR101" H 9600 850 50  0001 C CNN
 F 1 "GND" H 9600 950 50  0000 C CNN
 F 2 "" H 9600 1100 60  0000 C CNN
@@
 Connection ~ 9150 750
 $Comp
-L VCC #PWR098
+L VCC #PWR98
 U 1 1 56029609
 P 9150 700
-F 0 "#PWR098" H 9150 550 50  0001 C CNN
+F 0 "#PWR98" H 9150 550 50  0001 C CNN
 F 1 "VCC" H 9150 850 50  0000 C CNN
 F 2 "" H 9150 700 60  0000 C CNN
@@
 Connection ~ 8700 750
 $Comp
-L GND #PWR099
+L GND #PWR96
 U 1 1 5602C4DB
 P 8700 1100
-F 0 "#PWR099" H 8700 850 50  0001 C CNN
+F 0 "#PWR96" H 8700 850 50  0001 C CNN
 F 1 "GND" H 8700 950 50  0000 C CNN
 F 2 "" H 8700 1100 60  0000 C CNN
@@
 $EndComp
 $Comp
-L GND #PWR0100
+L GND #PWR95
 U 1 1 5602C537
 P 8400 1100
-F 0 "#PWR0100" H 8400 850 50  0001 C CNN
+F 0 "#PWR95" H 8400 850 50  0001 C CNN
 F 1 "GND" H 8400 950 50  0000 C CNN
 F 2 "" H 8400 1100 60  0000 C CNN
@@
 F 2 "CustomParts:C_0603_SM" H 10588 800 30  0001 C CNN
 F 3 "http://www.mouser.com/ds/2/447/UPY-GPHC_X7R_6.3V-to-50V_8-12304.pdf" H 10550 950 60  0001 C CNN
-F 4 "603-CC603KRX7R7BB105" H 10550 950 60  0001 C CNN "Mouse PN"
+F 4 "81-GRM188R71C105KA2J" H 10550 950 60  0001 C CNN "Mouse PN"
 	1    10550 950
 	1    0    0    -1
@@
 	9650 1800 9550 1800
 $Comp
-L GND #PWR0101
+L GND #PWR100
 U 1 1 56A15882
 P 9550 2100
-F 0 "#PWR0101" H 9550 1850 50  0001 C CNN
+F 0 "#PWR100" H 9550 1850 50  0001 C CNN
 F 1 "GND" H 9550 1950 50  0000 C CNN
 F 2 "" H 9550 2100 60  0000 C CNN
@@
 F 2 "Housings_QFP:TQFP-44_10x10mm_Pitch0.8mm" H 4250 2500 35  0001 C CIN
 F 3 "http://www.mouser.com/ds/2/36/Atmel-8387-8-and16-bit-AVR-Microcontroller-XMEGA-A-259135.pdf" H 4250 2500 60  0001 C CNN
-F 4 "556-ATXMEGA16A4U-AU" H 4250 2500 60  0001 C CNN "Mouse PN"
+F 4 "556-ATXMEGA128A4U-AU" H 4250 2500 60  0001 C CNN "Mouse PN"
 	1    4250 2500
 	1    0    0    -1
@@
 F 2 "Custom Parts:C_1206_SM" H 2150 2100 60  0001 C CNN
 F 3 "http://www.mouser.com/ds/2/360/SC-32P_Leaflet_r_newest-541780.pdf" H 2150 2100 60  0001 C CNN
-F 4 "628-SC32P-125PF20PPM" H 2150 2100 60  0001 C CNN "Mouser"
+F 4 "815-S07AIG-32.76891T" H 2150 2100 60  0001 C CNN "Mouser"
 	1    2150 2100
 	1    0    0    -1
@@
 	1850 2200 3350 2200
 $Comp
-L GND #PWR0102
+L GND #PWR92
 U 1 1 56DA1E3F
 P 2450 1800
-F 0 "#PWR0102" H 2450 1550 50  0001 C CNN
+F 0 "#PWR92" H 2450 1550 50  0001 C CNN
 F 1 "GND" H 2450 1650 50  0000 C CNN
 F 2 "" H 2450 1800 60  0000 C CNN
@@
 $EndComp
 $Comp
-L GND #PWR0103
+L GND #PWR91
 U 1 1 56DA2162
 P 1850 1800
-F 0 "#PWR0103" H 1850 1550 50  0001 C CNN
+F 0 "#PWR91" H 1850 1550 50  0001 C CNN
 F 1 "GND" H 1850 1650 50  0000 C CNN
 F 2 "" H 1850 1800 60  0000 C CNN

Commit message: Rev2.1 produced
Built R2.0, included findings, minor tweaks to placment and BOM.
Parts:
- C46: Mouse PN 81-GRM188R71C105KA2J -> 581-06036C105MAT2A
- C53, C54: Mouse PN 810-C1608C0G1H090C -> 81-GRM1885C1H9R0DA1D; Mouser DNS -> (none)
- R63: Mouse PN 71-CRCW0603-220-E3 -> 667-ERJ-3GEYJ221V
- X3: Mouse PN (none) -> 815-S07AIG-32.76891T; Mouser 815-S07AIG-32.76891T -> (none)
Changed lines of the file:
@@
 SEQ_LED2
 $Comp
-L GND #PWR93
+L GND #PWR090
 U 1 1 55F86E9C
 P 4100 3900
-F 0 "#PWR93" H 4100 3650 50  0001 C CNN
+F 0 "#PWR090" H 4100 3650 50  0001 C CNN
 F 1 "GND" H 4100 3750 50  0000 C CNN
 F 2 "" H 4100 3900 60  0000 C CNN
@@
 PDI
 $Comp
-L GND #PWR102
+L GND #PWR091
 U 1 1 55F86EF0
 P 10000 3650
-F 0 "#PWR102" H 10000 3400 50  0001 C CNN
+F 0 "#PWR091" H 10000 3400 50  0001 C CNN
 F 1 "GND" H 10000 3500 50  0000 C CNN
 F 2 "" H 10000 3650 60  0000 C CNN
@@
 5V0_B_EN
 $Comp
-L GND #PWR90
+L GND #PWR092
 U 1 1 55FA434A
 P 1600 7100
-F 0 "#PWR90" H 1600 6850 50  0001 C CNN
+F 0 "#PWR092" H 1600 6850 50  0001 C CNN
 F 1 "GND" H 1600 6950 50  0000 C CNN
 F 2 "" H 1600 7100 60  0000 C CNN
@@
 $EndComp
 $Comp
-L GND #PWR94
+L GND #PWR093
 U 1 1 55FE1020
 P 6400 5050
-F 0 "#PWR94" H 6400 4800 50  0001 C CNN
+F 0 "#PWR093" H 6400 4800 50  0001 C CNN
 F 1 "GND" H 6400 4900 50  0000 C CNN
 F 2 "" H 6400 5050 60  0000 C CNN
@@
 Connection ~ 10550 750
 $Comp
-L GND #PWR103
+L GND #PWR094
 U 1 1 56006FBB
 P 10550 1100
-F 0 "#PWR103" H 10550 850 50  0001 C CNN
+F 0 "#PWR094" H 10550 850 50  0001 C CNN
 F 1 "GND" H 10550 950 50  0000 C CNN
 F 2 "" H 10550 1100 60  0000 C CNN
@@
 Connection ~ 9000 750
 $Comp
-L GND #PWR97
+L GND #PWR095
 U 1 1 560285A0
 P 9000 1100
-F 0 "#PWR97" H 9000 850 50  0001 C CNN
+F 0 "#PWR095" H 9000 850 50  0001 C CNN
 F 1 "GND" H 9000 950 50  0000 C CNN
 F 2 "" H 9000 1100 60  0000 C CNN
@@
 $EndComp
 $Comp
-L GND #PWR99
+L GND #PWR096
 U 1 1 560285F6
 P 9300 1100
-F 0 "#PWR99" H 9300 850 50  0001 C CNN
+F 0 "#PWR096" H 9300 850 50  0001 C CNN
 F 1 "GND" H 9300 950 50  0000 C CNN
 F 2 "" H 9300 1100 60  0000 C CNN
@@
 $EndComp
 $Comp
-L GND #PWR101
+L GND #PWR097
 U 1 1 5602864C
 P 9600 1100
-F 0 "#PWR101" H 9600 850 50  0001 C CNN
+F 0 "#PWR097" H 9600 850 50  0001 C CNN
 F 1 "GND" H 9600 950 50  0000 C CNN
 F 2 "" H 9600 1100 60  0000 C CNN
@@
 Connection ~ 9150 750
 $Comp
-L VCC #PWR98
+L VCC #PWR098
 U 1 1 56029609
 P 9150 700
-F 0 "#PWR98" H 9150 550 50  0001 C CNN
+F 0 "#PWR098" H 9150 550 50  0001 C CNN
 F 1 "VCC" H 9150 850 50  0000 C CNN
 F 2 "" H 9150 700 60  0000 C CNN
@@
 Connection ~ 8700 750
 $Comp
-L GND #PWR96
+L GND #PWR099
 U 1 1 5602C4DB
 P 8700 1100
-F 0 "#PWR96" H 8700 850 50  0001 C CNN
+F 0 "#PWR099" H 8700 850 50  0001 C CNN
 F 1 "GND" H 8700 950 50  0000 C CNN
 F 2 "" H 8700 1100 60  0000 C CNN
@@
 $EndComp
 $Comp
-L GND #PWR95
+L GND #PWR0100
 U 1 1 5602C537
 P 8400 1100
-F 0 "#PWR95" H 8400 850 50  0001 C CNN
+F 0 "#PWR0100" H 8400 850 50  0001 C CNN
 F 1 "GND" H 8400 950 50  0000 C CNN
 F 2 "" H 8400 1100 60  0000 C CNN
@@
 F 2 "CustomParts:C_0603_SM" H 10588 800 30  0001 C CNN
 F 3 "http://www.mouser.com/ds/2/447/UPY-GPHC_X7R_6.3V-to-50V_8-12304.pdf" H 10550 950 60  0001 C CNN
-F 4 "81-GRM188R71C105KA2J" H 10550 950 60  0001 C CNN "Mouse PN"
+F 4 "581-06036C105MAT2A" H 10550 950 60  0001 C CNN "Mouse PN"
 	1    10550 950
 	1    0    0    -1
@@
 F 2 "CustomParts:R_0603_sm" V 9730 5050 30  0001 C CNN
 F 3 "http://www.mouser.com/ds/2/427/dcrcwe3-109170.pdf" H 9800 5050 30  0001 C CNN
-F 4 "71-CRCW0603-220-E3" H 9800 5050 60  0001 C CNN "Mouse PN"
+F 4 "667-ERJ-3GEYJ221V" H 9800 5050 60  0001 C CNN "Mouse PN"
 	1    9800 5050
 	-1   0    0    1
@@
 	9650 1800 9550 1800
 $Comp
-L GND #PWR100
+L GND #PWR0101
 U 1 1 56A15882
 P 9550 2100
-F 0 "#PWR100" H 9550 1850 50  0001 C CNN
+F 0 "#PWR0101" H 9550 1850 50  0001 C CNN
 F 1 "GND" H 9550 1950 50  0000 C CNN
 F 2 "" H 9550 2100 60  0000 C CNN
@@
 F 2 "Custom Parts:C_1206_SM" H 2150 2100 60  0001 C CNN
 F 3 "http://www.mouser.com/ds/2/360/SC-32P_Leaflet_r_newest-541780.pdf" H 2150 2100 60  0001 C CNN
-F 4 "815-S07AIG-32.76891T" H 2150 2100 60  0001 C CNN "Mouser"
+F 4 "815-S07AIG-32.76891T" H 2150 2100 60  0001 C CNN "Mouse PN"
 	1    2150 2100
 	1    0    0    -1
@@
 F 1 "9p" H 1875 1850 50  0000 L CNN
 F 2 "CustomParts:C_0603_SM" H 1888 1800 30  0001 C CNN
-F 3 "http://www.mouser.com/ds/2/400/lcc_commercial_general_en-837201.pdf" H 1850 1950 60  0001 C CNN
-F 4 "DNS" H 1850 1950 60  0001 C CNN "Mouser"
-F 5 "810-C1608C0G1H090C" H 1850 1950 60  0001 C CNN "Mouse PN"
+F 3 "http://www.mouser.com/ds/2/281/c02e-2905.pdf" H 1850 1950 60  0001 C CNN
+F 4 "81-GRM1885C1H9R0DA1D" H 1850 1950 60  0001 C CNN "Mouse PN"
 	1    1850 1950
 	-1   0    0    -1
@@
 F 1 "9p" H 2475 1850 50  0000 L CNN
 F 2 "CustomParts:C_0603_SM" H 2488 1800 30  0001 C CNN
-F 3 "http://www.mouser.com/ds/2/400/lcc_commercial_general_en-837201.pdf" H 2450 1950 60  0001 C CNN
-F 4 "DNS" H 2450 1950 60  0001 C CNN "Mouser"
-F 5 "810-C1608C0G1H090C" H 2450 1950 60  0001 C CNN "Mouse PN"
+F 3 "http://www.mouser.com/ds/2/281/c02e-2905.pdf" H 2450 1950 60  0001 C CNN
+F 4 "81-GRM1885C1H9R0DA1D" H 2450 1950 60  0001 C CNN "Mouse PN"
 	1    2450 1950
 	-1   0    0    -1
@@
 	1850 2200 3350 2200
 $Comp
-L GND #PWR92
+L GND #PWR0102
 U 1 1 56DA1E3F
 P 2450 1800
-F 0 "#PWR92" H 2450 1550 50  0001 C CNN
+F 0 "#PWR0102" H 2450 1550 50  0001 C CNN
 F 1 "GND" H 2450 1650 50  0000 C CNN
 F 2 "" H 2450 1800 60  0000 C CNN
@@
 $EndComp
 $Comp
-L GND #PWR91
+L GND #PWR0103
 U 1 1 56DA2162
 P 1850 1800
-F 0 "#PWR91" H 1850 1550 50  0001 C CNN
+F 0 "#PWR0103" H 1850 1550 50  0001 C CNN
 F 1 "GND" H 1850 1650 50  0000 C CNN
 F 2 "" H 1850 1800 60  0000 C CNN
