File: MakeFiles/V2X_GSM.sch (KiCad schematic (older format))
At the start: 44 parts, among them P1 SIM_SKT, P14 CUR_SEN, P2 SMA, P26 CONN_02X10, P3 SMA, Q12 IRF9335, U13 XRP6124, U24 TLV70012DCK, U3 MMQA5V6T3G, U4 SIM5320

Commit message: 53851 Import of V2X R2.0
capture from legacy repo
Parts:
- removed C15, C46: 330P, Custom Parts:C_0603_SM, symbol C
- removed C19, C25: 100N, Custom Parts:C_0603_SM, symbol C
- removed C20, C24, C28, C47: 4U7, Custom Parts:C_0805_SM, symbol C
- removed C23, C26: 220U, Capacitors_SMD:c_elec_6.3x5.8, symbol CP
- removed C27: 10N, Custom Parts:C_0603_SM, symbol C
- removed C48, C49: 10U, Custom Parts:C_1206_SM, symbol C
- removed D3: SBR3U30P1-7, Diodes_SMD:SOD-123, symbol D_Schottky_Small
- removed FB3: 220, Custom Parts:R_0603_sm, symbol FILTER
- removed L4: 5U6, Custom Parts:4.5x4.5mm_Ind, symbol INDUCTOR_SMALL
- removed P14: CUR_SEN, Connect:PINHEAD1-2, symbol CONN_01X02
- removed P26: CONN_02X10, Pin_Headers:Pin_Header_Straight_2x10, symbol CONN_02X10
- removed Q12: IRF9335, Custom Parts:SOIC-8_MOS, symbol Q_PMOS_GSD
- removed R16: 2K0, Custom Parts:R_0603_sm, symbol R
- removed R17: 8K2, Custom Parts:R_0603_sm, symbol R
- removed R8, R84, R86, R9: DNS, Custom Parts:R_0603_sm, symbol R
- removed R85: 0, Custom Parts:R_0603_sm, symbol R
- removed U13: XRP6124, Housings_SOT-23_SOT-143_TSOT-6:SOT-23-5, symbol XRP6124
- removed U24: TLV70012DCK, symbol TLV70012DCK
- C48: renamed from C17; footprint Custom Parts:C_0603_SM -> CustomParts:C_0603_SM
- C49: renamed from C14; footprint Custom Parts:C_0603_SM -> CustomParts:C_0603_SM
- C50: renamed from C18; footprint Custom Parts:C_0603_SM -> CustomParts:C_0603_SM
- C51: renamed from C21; footprint Custom Parts:C_0603_SM -> CustomParts:C_0603_SM
- L3: renamed from L2; footprint Custom Parts:C_0603_SM -> CustomParts:L_0603_SM
- L4: renamed from L1; footprint Custom Parts:C_0603_SM -> CustomParts:L_0603_SM
- P22: renamed from P2; footprint Custom Parts:SMA-RA_142-0701-801 -> CustomParts:SMA-RA_142-0701-801
- P23: renamed from P3; footprint Custom Parts:SMA-RA_142-0701-801 -> CustomParts:SMA-RA_142-0701-801
- P24: renamed from P1; footprint Custom Parts:47553-1001 -> CustomParts:47553-1001
- R69: renamed from R13; footprint Custom Parts:R_0603_sm -> CustomParts:R_0603_sm
- R70: renamed from R12; footprint Custom Parts:R_0603_sm -> CustomParts:R_0603_sm
- R71: renamed from R14; footprint Custom Parts:R_0603_sm -> CustomParts:R_0603_sm
- U22: renamed from U4; footprint Custom Parts:SIM5320 -> CustomParts:SIM5320
- U23: renamed from U3; footprint Housings_SOT-23_SOT-143_TSOT-6:SOT-23-6 -> TO_SOT_Packages_SMD:SOT-23-6
- renumbered C16 to C47, W2 to W1
Connections:
- net labels added: 4V1, GPS_EN, HUB_PWR_PRT2, SEQ_WAKE, SIMCARD, SIM_DM, SIM_DP, SIM_NET, SIM_RESET, SIM_RXD, SIM_TXD, SIM_WAKE, ~SIM_PWR_ON
- net labels removed: 12V0_C, 4V1_B, 4V1_EN_B, PC_WAKE, SIMCARD_B, SIM_DM_B, SIM_DP_B, SIM_DTR, SIM_NET_B, SIM_PWR_B, SIM_PWR_ON_B, SIM_RESET_B, SIM_RF_OFF_B, SIM_RI, SIM_RXD_B, SIM_TXD_B, SIM_USB_DET_B, SIM_WAKE_B
- wire segments 63 -> 24
- no-connect marks 38 -> 41
Other:
- note removed: "4.1V @ 1.5A DC-DC Power Supply"
- note removed: "Hopefully the PWRCTRL can \nmomentarily use a pull up \nresistor to snense the card,\n otherwise resistors"
- note removed: "SIM side"
- moved on the sheet: C48, C49, C50, C51, L3, L4, P22, P23, U23, W1

Commit message: Part numer updates
for error or out of stock
Parts:
- C51: footprint CustomParts:C_0603_SM -> CustomParts:C_0805_SM
Changed lines of the file:
@@
 $EndDescr
 $Comp
-L GND #PWR0104
+L GND #PWR104
 U 1 1 55A6AD93
 P 1950 1650
-F 0 "#PWR0104" H 1950 1400 50  0001 C CNN
+F 0 "#PWR104" H 1950 1400 50  0001 C CNN
 F 1 "GND" H 1950 1500 50  0000 C CNN
 F 2 "" H 1950 1650 60  0000 C CNN
@@
 $EndComp
 $Comp
-L GND #PWR0105
+L GND #PWR105
 U 1 1 55A6ADB3
 P 1950 1750
-F 0 "#PWR0105" H 1950 1500 50  0001 C CNN
+F 0 "#PWR105" H 1950 1500 50  0001 C CNN
 F 1 "GND" H 1950 1600 50  0000 C CNN
 F 2 "" H 1950 1750 60  0000 C CNN
@@
 $EndComp
 $Comp
-L GND #PWR0106
+L GND #PWR106
 U 1 1 55A6ADC8
 P 1950 2050
-F 0 "#PWR0106" H 1950 1800 50  0001 C CNN
+F 0 "#PWR106" H 1950 1800 50  0001 C CNN
 F 1 "GND" H 1950 1900 50  0000 C CNN
 F 2 "" H 1950 2050 60  0000 C CNN
@@
 $EndComp
 $Comp
-L GND #PWR0107
+L GND #PWR107
 U 1 1 55A6ADD6
 P 1950 2550
-F 0 "#PWR0107" H 1950 2300 50  0001 C CNN
+F 0 "#PWR107" H 1950 2300 50  0001 C CNN
 F 1 "GND" H 1950 2400 50  0000 C CNN
 F 2 "" H 1950 2550 60  0000 C CNN
@@
 $EndComp
 $Comp
-L GND #PWR0108
+L GND #PWR108
 U 1 1 55A6AE04
 P 1950 2950
-F 0 "#PWR0108" H 1950 2700 50  0001 C CNN
+F 0 "#PWR108" H 1950 2700 50  0001 C CNN
 F 1 "GND" H 1950 2800 50  0000 C CNN
 F 2 "" H 1950 2950 60  0000 C CNN
@@
 $EndComp
 $Comp
-L GND #PWR0109
+L GND #PWR114
 U 1 1 55A6AE12
 P 4050 4050
-F 0 "#PWR0109" H 4050 3800 50  0001 C CNN
+F 0 "#PWR114" H 4050 3800 50  0001 C CNN
 F 1 "GND" H 4050 3900 50  0000 C CNN
 F 2 "" H 4050 4050 60  0000 C CNN
@@
 $EndComp
 $Comp
-L GND #PWR0110
+L GND #PWR116
 U 1 1 55A6AE37
 P 4350 4050
-F 0 "#PWR0110" H 4350 3800 50  0001 C CNN
+F 0 "#PWR116" H 4350 3800 50  0001 C CNN
 F 1 "GND" H 4350 3900 50  0000 C CNN
 F 2 "" H 4350 4050 60  0000 C CNN
@@
 $EndComp
 $Comp
-L GND #PWR0111
+L GND #PWR121
 U 1 1 55A6AE45
 P 4850 3550
-F 0 "#PWR0111" H 4850 3300 50  0001 C CNN
+F 0 "#PWR121" H 4850 3300 50  0001 C CNN
 F 1 "GND" H 4850 3400 50  0000 C CNN
 F 2 "" H 4850 3550 60  0000 C CNN
@@
 $EndComp
 $Comp
-L GND #PWR0112
+L GND #PWR120
 U 1 1 55A6AE61
 P 4850 3350
-F 0 "#PWR0112" H 4850 3100 50  0001 C CNN
+F 0 "#PWR120" H 4850 3100 50  0001 C CNN
 F 1 "GND" H 4850 3200 50  0000 C CNN
 F 2 "" H 4850 3350 60  0000 C CNN
@@
 $EndComp
 $Comp
-L GND #PWR0113
+L GND #PWR117
 U 1 1 55A6AE6F
 P 4850 1650
-F 0 "#PWR0113" H 4850 1400 50  0001 C CNN
+F 0 "#PWR117" H 4850 1400 50  0001 C CNN
 F 1 "GND" H 4850 1500 50  0000 C CNN
 F 2 "" H 4850 1650 60  0000 C CNN
@@
 $EndComp
 $Comp
-L GND #PWR0114
+L GND #PWR118
 U 1 1 55A6AE7D
 P 4850 1850
-F 0 "#PWR0114" H 4850 1600 50  0001 C CNN
+F 0 "#PWR118" H 4850 1600 50  0001 C CNN
 F 1 "GND" H 4850 1700 50  0000 C CNN
 F 2 "" H 4850 1850 60  0000 C CNN
@@
 $EndComp
 $Comp
-L GND #PWR0115
+L GND #PWR119
 U 1 1 55A6AE8B
 P 4850 1950
-F 0 "#PWR0115" H 4850 1700 50  0001 C CNN
+F 0 "#PWR119" H 4850 1700 50  0001 C CNN
 F 1 "GND" H 4850 1800 50  0000 C CNN
 F 2 "" H 4850 1950 60  0000 C CNN
@@
 $EndComp
 $Comp
-L GND #PWR0116
+L GND #PWR115
 U 1 1 55A6AE99
 P 4350 1150
-F 0 "#PWR0116" H 4350 900 50  0001 C CNN
+F 0 "#PWR115" H 4350 900 50  0001 C CNN
 F 1 "GND" H 4350 1000 50  0000 C CNN
 F 2 "" H 4350 1150 60  0000 C CNN
@@
 $EndComp
 $Comp
-L GND #PWR0117
+L GND #PWR113
 U 1 1 55A6AEA7
 P 4050 1150
-F 0 "#PWR0117" H 4050 900 50  0001 C CNN
+F 0 "#PWR113" H 4050 900 50  0001 C CNN
 F 1 "GND" H 4050 1000 50  0000 C CNN
 F 2 "" H 4050 1150 60  0000 C CNN
@@
 $EndComp
 $Comp
-L GND #PWR0118
+L GND #PWR112
 U 1 1 55A6AEB5
 P 3950 1150
-F 0 "#PWR0118" H 3950 900 50  0001 C CNN
+F 0 "#PWR112" H 3950 900 50  0001 C CNN
 F 1 "GND" H 3950 1000 50  0000 C CNN
 F 2 "" H 3950 1150 60  0000 C CNN
@@
 $EndComp
 $Comp
-L GND #PWR0119
+L GND #PWR111
 U 1 1 55A6AEC3
 P 2750 1150
-F 0 "#PWR0119" H 2750 900 50  0001 C CNN
+F 0 "#PWR111" H 2750 900 50  0001 C CNN
 F 1 "GND" H 2750 1000 50  0000 C CNN
 F 2 "" H 2750 1150 60  0000 C CNN
@@
 $EndComp
 $Comp
-L GND #PWR0120
+L GND #PWR110
 U 1 1 55A6AED1
 P 2650 1150
-F 0 "#PWR0120" H 2650 900 50  0001 C CNN
+F 0 "#PWR110" H 2650 900 50  0001 C CNN
 F 1 "GND" H 2650 1000 50  0000 C CNN
 F 2 "" H 2650 1150 60  0000 C CNN
@@
 $EndComp
 $Comp
-L GND #PWR0121
+L GND #PWR109
 U 1 1 55A6AEDF
 P 2450 1150
-F 0 "#PWR0121" H 2450 900 50  0001 C CNN
+F 0 "#PWR109" H 2450 900 50  0001 C CNN
 F 1 "GND" H 2450 1000 50  0000 C CNN
 F 2 "" H 2450 1150 60  0000 C CNN
@@
 $EndComp
 $Comp
-L GND #PWR0122
+L GND #PWR130
 U 1 1 55A75A03
 P 9650 900
-F 0 "#PWR0122" H 9650 650 50  0001 C CNN
+F 0 "#PWR130" H 9650 650 50  0001 C CNN
 F 1 "GND" H 9650 750 50  0000 C CNN
 F 2 "" H 9650 900 60  0000 C CNN
@@
 $EndComp
 $Comp
-L GND #PWR0123
+L GND #PWR132
 U 1 1 55A75A4D
 P 9650 1800
-F 0 "#PWR0123" H 9650 1550 50  0001 C CNN
+F 0 "#PWR132" H 9650 1550 50  0001 C CNN
 F 1 "GND" H 9650 1650 50  0000 C CNN
 F 2 "" H 9650 1800 60  0000 C CNN
@@
 SIMCARD_V
 $Comp
-L GND #PWR0124
+L GND #PWR131
 U 1 1 55A75BB0
 P 9650 1300
-F 0 "#PWR0124" H 9650 1050 50  0001 C CNN
+F 0 "#PWR131" H 9650 1050 50  0001 C CNN
 F 1 "GND" H 9650 1150 50  0000 C CNN
 F 2 "" H 9650 1300 60  0000 C CNN
@@
 $EndComp
 $Comp
-L GND #PWR0125
+L GND #PWR126
 U 1 1 55A784DB
 P 7200 2150
-F 0 "#PWR0125" H 7200 1900 50  0001 C CNN
+F 0 "#PWR126" H 7200 1900 50  0001 C CNN
 F 1 "GND" H 7200 2000 50  0000 C CNN
 F 2 "" H 7200 2150 60  0000 C CNN
@@
 SIM Card
 $Comp
-L GND #PWR0126
+L GND #PWR123
 U 1 1 55A7D4E3
 P 6800 4050
-F 0 "#PWR0126" H 6800 3800 50  0001 C CNN
+F 0 "#PWR123" H 6800 3800 50  0001 C CNN
 F 1 "GND" H 6800 3900 50  0000 C CNN
 F 2 "" H 6800 4050 60  0000 C CNN
@@
 $EndComp
 $Comp
-L GND #PWR0127
+L GND #PWR128
 U 1 1 55A84AE6
 P 7950 1300
-F 0 "#PWR0127" H 7950 1050 50  0001 C CNN
+F 0 "#PWR128" H 7950 1050 50  0001 C CNN
 F 1 "GND" H 7950 1150 50  0000 C CNN
 F 2 "" H 7950 1300 60  0000 C CNN
@@
 $EndComp
 $Comp
-L GND #PWR0128
+L GND #PWR122
 U 1 1 55A92AA3
 P 5200 3750
-F 0 "#PWR0128" H 5200 3500 50  0001 C CNN
+F 0 "#PWR122" H 5200 3500 50  0001 C CNN
 F 1 "GND" H 5200 3600 50  0000 C CNN
 F 2 "" H 5200 3750 60  0000 C CNN
@@
 $EndComp
 $Comp
-L GND #PWR0129
+L GND #PWR124
 U 1 1 55A9AF9B
 P 7050 3500
-F 0 "#PWR0129" H 7050 3250 50  0001 C CNN
+F 0 "#PWR124" H 7050 3250 50  0001 C CNN
 F 1 "GND" H 7050 3350 50  0000 C CNN
 F 2 "" H 7050 3500 60  0000 C CNN
@@
 $EndComp
 $Comp
-L GND #PWR0130
+L GND #PWR127
 U 1 1 55A9B051
 P 7300 3500
-F 0 "#PWR0130" H 7300 3250 50  0001 C CNN
+F 0 "#PWR127" H 7300 3250 50  0001 C CNN
 F 1 "GND" H 7300 3350 50  0000 C CNN
 F 2 "" H 7300 3500 60  0000 C CNN
@@
 $EndComp
 $Comp
-L GND #PWR0131
+L GND #PWR129
 U 1 1 55A9FAF5
 P 9300 3600
-F 0 "#PWR0131" H 9300 3350 50  0001 C CNN
+F 0 "#PWR129" H 9300 3350 50  0001 C CNN
 F 1 "GND" H 9300 3450 50  0000 C CNN
 F 2 "" H 9300 3600 60  0000 C CNN
@@
 $EndComp
 $Comp
-L GND #PWR0132
+L GND #PWR125
 U 1 1 56099B91
 P 7150 1300
-F 0 "#PWR0132" H 7150 1050 50  0001 C CNN
+F 0 "#PWR125" H 7150 1050 50  0001 C CNN
 F 1 "GND" H 7150 1150 50  0000 C CNN
 F 2 "" H 7150 1300 60  0000 C CNN
@@
 F 0 "C51" H 7325 4050 50  0000 L CNN
 F 1 "150p" H 7325 3850 50  0000 L CNN
-F 2 "CustomParts:C_0603_SM" H 7338 3800 30  0001 C CNN
+F 2 "CustomParts:C_0805_SM" H 7338 3800 30  0001 C CNN
 F 3 "http://www.mouser.com/ds/2/427/highq-222791.pdf" H 7300 3950 60  0001 C CNN
 F 4 "77-VJ0805Q151JXAAC" H 7300 3950 60  0001 C CNN "Mouse PN"

Commit message: Rev2.1 produced
Built R2.0, included findings, minor tweaks to placment and BOM.
Parts:
- C47: Mouse PN (none) -> 504-KR-5R5C104-R; Mouser PN 504-KR-5R5C104-R -> (none)
- C48: Mouse PN 581-08052U560G -> 77-VJ0603A560JXACBC
- U22: AliExpress PN SIM5320A -> (none); Mouse PN # -> AliExpressOrder
Changed lines of the file:
@@
 $EndDescr
 $Comp
-L GND #PWR104
+L GND #PWR0104
 U 1 1 55A6AD93
 P 1950 1650
-F 0 "#PWR104" H 1950 1400 50  0001 C CNN
+F 0 "#PWR0104" H 1950 1400 50  0001 C CNN
 F 1 "GND" H 1950 1500 50  0000 C CNN
 F 2 "" H 1950 1650 60  0000 C CNN
@@
 $EndComp
 $Comp
-L GND #PWR105
+L GND #PWR0105
 U 1 1 55A6ADB3
 P 1950 1750
-F 0 "#PWR105" H 1950 1500 50  0001 C CNN
+F 0 "#PWR0105" H 1950 1500 50  0001 C CNN
 F 1 "GND" H 1950 1600 50  0000 C CNN
 F 2 "" H 1950 1750 60  0000 C CNN
@@
 $EndComp
 $Comp
-L GND #PWR106
+L GND #PWR0106
 U 1 1 55A6ADC8
 P 1950 2050
-F 0 "#PWR106" H 1950 1800 50  0001 C CNN
+F 0 "#PWR0106" H 1950 1800 50  0001 C CNN
 F 1 "GND" H 1950 1900 50  0000 C CNN
 F 2 "" H 1950 2050 60  0000 C CNN
@@
 $EndComp
 $Comp
-L GND #PWR107
+L GND #PWR0107
 U 1 1 55A6ADD6
 P 1950 2550
-F 0 "#PWR107" H 1950 2300 50  0001 C CNN
+F 0 "#PWR0107" H 1950 2300 50  0001 C CNN
 F 1 "GND" H 1950 2400 50  0000 C CNN
 F 2 "" H 1950 2550 60  0000 C CNN
@@
 $EndComp
 $Comp
-L GND #PWR108
+L GND #PWR0108
 U 1 1 55A6AE04
 P 1950 2950
-F 0 "#PWR108" H 1950 2700 50  0001 C CNN
+F 0 "#PWR0108" H 1950 2700 50  0001 C CNN
 F 1 "GND" H 1950 2800 50  0000 C CNN
 F 2 "" H 1950 2950 60  0000 C CNN
@@
 $EndComp
 $Comp
-L GND #PWR114
+L GND #PWR0109
 U 1 1 55A6AE12
 P 4050 4050
-F 0 "#PWR114" H 4050 3800 50  0001 C CNN
+F 0 "#PWR0109" H 4050 3800 50  0001 C CNN
 F 1 "GND" H 4050 3900 50  0000 C CNN
 F 2 "" H 4050 4050 60  0000 C CNN
@@
 $EndComp
 $Comp
-L GND #PWR116
+L GND #PWR0110
 U 1 1 55A6AE37
 P 4350 4050
-F 0 "#PWR116" H 4350 3800 50  0001 C CNN
+F 0 "#PWR0110" H 4350 3800 50  0001 C CNN
 F 1 "GND" H 4350 3900 50  0000 C CNN
 F 2 "" H 4350 4050 60  0000 C CNN
@@
 $EndComp
 $Comp
-L GND #PWR121
+L GND #PWR0111
 U 1 1 55A6AE45
 P 4850 3550
-F 0 "#PWR121" H 4850 3300 50  0001 C CNN
+F 0 "#PWR0111" H 4850 3300 50  0001 C CNN
 F 1 "GND" H 4850 3400 50  0000 C CNN
 F 2 "" H 4850 3550 60  0000 C CNN
@@
 $EndComp
 $Comp
-L GND #PWR120
+L GND #PWR0112
 U 1 1 55A6AE61
 P 4850 3350
-F 0 "#PWR120" H 4850 3100 50  0001 C CNN
+F 0 "#PWR0112" H 4850 3100 50  0001 C CNN
 F 1 "GND" H 4850 3200 50  0000 C CNN
 F 2 "" H 4850 3350 60  0000 C CNN
@@
 $EndComp
 $Comp
-L GND #PWR117
+L GND #PWR0113
 U 1 1 55A6AE6F
 P 4850 1650
-F 0 "#PWR117" H 4850 1400 50  0001 C CNN
+F 0 "#PWR0113" H 4850 1400 50  0001 C CNN
 F 1 "GND" H 4850 1500 50  0000 C CNN
 F 2 "" H 4850 1650 60  0000 C CNN
@@
 $EndComp
 $Comp
-L GND #PWR118
+L GND #PWR0114
 U 1 1 55A6AE7D
 P 4850 1850
-F 0 "#PWR118" H 4850 1600 50  0001 C CNN
+F 0 "#PWR0114" H 4850 1600 50  0001 C CNN
 F 1 "GND" H 4850 1700 50  0000 C CNN
 F 2 "" H 4850 1850 60  0000 C CNN
@@
 $EndComp
 $Comp
-L GND #PWR119
+L GND #PWR0115
 U 1 1 55A6AE8B
 P 4850 1950
-F 0 "#PWR119" H 4850 1700 50  0001 C CNN
+F 0 "#PWR0115" H 4850 1700 50  0001 C CNN
 F 1 "GND" H 4850 1800 50  0000 C CNN
 F 2 "" H 4850 1950 60  0000 C CNN
@@
 $EndComp
 $Comp
-L GND #PWR115
+L GND #PWR0116
 U 1 1 55A6AE99
 P 4350 1150
-F 0 "#PWR115" H 4350 900 50  0001 C CNN
+F 0 "#PWR0116" H 4350 900 50  0001 C CNN
 F 1 "GND" H 4350 1000 50  0000 C CNN
 F 2 "" H 4350 1150 60  0000 C CNN
@@
 $EndComp
 $Comp
-L GND #PWR113
+L GND #PWR0117
 U 1 1 55A6AEA7
 P 4050 1150
-F 0 "#PWR113" H 4050 900 50  0001 C CNN
+F 0 "#PWR0117" H 4050 900 50  0001 C CNN
 F 1 "GND" H 4050 1000 50  0000 C CNN
 F 2 "" H 4050 1150 60  0000 C CNN
@@
 $EndComp
 $Comp
-L GND #PWR112
+L GND #PWR0118
 U 1 1 55A6AEB5
 P 3950 1150
-F 0 "#PWR112" H 3950 900 50  0001 C CNN
+F 0 "#PWR0118" H 3950 900 50  0001 C CNN
 F 1 "GND" H 3950 1000 50  0000 C CNN
 F 2 "" H 3950 1150 60  0000 C CNN
@@
 $EndComp
 $Comp
-L GND #PWR111
+L GND #PWR0119
 U 1 1 55A6AEC3
 P 2750 1150
-F 0 "#PWR111" H 2750 900 50  0001 C CNN
+F 0 "#PWR0119" H 2750 900 50  0001 C CNN
 F 1 "GND" H 2750 1000 50  0000 C CNN
 F 2 "" H 2750 1150 60  0000 C CNN
@@
 $EndComp
 $Comp
-L GND #PWR110
+L GND #PWR0120
 U 1 1 55A6AED1
 P 2650 1150
-F 0 "#PWR110" H 2650 900 50  0001 C CNN
+F 0 "#PWR0120" H 2650 900 50  0001 C CNN
 F 1 "GND" H 2650 1000 50  0000 C CNN
 F 2 "" H 2650 1150 60  0000 C CNN
@@
 $EndComp
 $Comp
-L GND #PWR109
+L GND #PWR0121
 U 1 1 55A6AEDF
 P 2450 1150
-F 0 "#PWR109" H 2450 900 50  0001 C CNN
+F 0 "#PWR0121" H 2450 900 50  0001 C CNN
 F 1 "GND" H 2450 1000 50  0000 C CNN
 F 2 "" H 2450 1150 60  0000 C CNN
@@
 $EndComp
 $Comp
-L GND #PWR130
+L GND #PWR0122
 U 1 1 55A75A03
 P 9650 900
-F 0 "#PWR130" H 9650 650 50  0001 C CNN
+F 0 "#PWR0122" H 9650 650 50  0001 C CNN
 F 1 "GND" H 9650 750 50  0000 C CNN
 F 2 "" H 9650 900 60  0000 C CNN
@@
 $EndComp
 $Comp
-L GND #PWR132
+L GND #PWR0123
 U 1 1 55A75A4D
 P 9650 1800
-F 0 "#PWR132" H 9650 1550 50  0001 C CNN
+F 0 "#PWR0123" H 9650 1550 50  0001 C CNN
 F 1 "GND" H 9650 1650 50  0000 C CNN
 F 2 "" H 9650 1800 60  0000 C CNN
@@
 SIMCARD_V
 $Comp
-L GND #PWR131
+L GND #PWR0124
 U 1 1 55A75BB0
 P 9650 1300
-F 0 "#PWR131" H 9650 1050 50  0001 C CNN
+F 0 "#PWR0124" H 9650 1050 50  0001 C CNN
 F 1 "GND" H 9650 1150 50  0000 C CNN
 F 2 "" H 9650 1300 60  0000 C CNN
@@
 $EndComp
 $Comp
-L GND #PWR126
+L GND #PWR0125
 U 1 1 55A784DB
 P 7200 2150
-F 0 "#PWR126" H 7200 1900 50  0001 C CNN
+F 0 "#PWR0125" H 7200 1900 50  0001 C CNN
 F 1 "GND" H 7200 2000 50  0000 C CNN
 F 2 "" H 7200 2150 60  0000 C CNN
@@
 SIM Card
 $Comp
-L GND #PWR123
+L GND #PWR0126
 U 1 1 55A7D4E3
 P 6800 4050
-F 0 "#PWR123" H 6800 3800 50  0001 C CNN
+F 0 "#PWR0126" H 6800 3800 50  0001 C CNN
 F 1 "GND" H 6800 3900 50  0000 C CNN
 F 2 "" H 6800 4050 60  0000 C CNN
@@
 $EndComp
 $Comp
-L GND #PWR128
+L GND #PWR0127
 U 1 1 55A84AE6
 P 7950 1300
-F 0 "#PWR128" H 7950 1050 50  0001 C CNN
+F 0 "#PWR0127" H 7950 1050 50  0001 C CNN
 F 1 "GND" H 7950 1150 50  0000 C CNN
 F 2 "" H 7950 1300 60  0000 C CNN
@@
 F 2 "Capacitors_ThroughHole:C_Radial_D12.5_L25_P5" H 5200 3600 60  0001 C CNN
 F 3 "http://www.mouser.com/ds/2/87/Bus_Elx_DS_4327_KR_Series-479311.pdf" H 5200 3600 60  0001 C CNN
-F 4 "504-KR-5R5C104-R" H 5200 3600 60  0001 C CNN "Mouser PN"
+F 4 "504-KR-5R5C104-R" H 5200 3600 60  0001 C CNN "Mouse PN"
 	1    5200 3600
 	1    0    0    -1
 $EndComp
 $Comp
-L GND #PWR122
+L GND #PWR0128
 U 1 1 55A92AA3
 P 5200 3750
-F 0 "#PWR122" H 5200 3500 50  0001 C CNN
+F 0 "#PWR0128" H 5200 3500 50  0001 C CNN
 F 1 "GND" H 5200 3600 50  0000 C CNN
 F 2 "" H 5200 3750 60  0000 C CNN
@@
 F 1 "56P" H 7075 3250 50  0000 L CNN
 F 2 "CustomParts:C_0603_SM" H 7088 3200 30  0001 C CNN
-F 3 "http://www.mouser.com/ds/2/40/useries-37712.pdf" H 7050 3350 60  0001 C CNN
-F 4 "581-08052U560G" H 7050 3350 60  0001 C CNN "Mouse PN"
+F 3 "http://www.mouser.com/ds/2/427/vjw1bcbascomseries-223529.pdf" H 7050 3350 60  0001 C CNN
+F 4 "77-VJ0603A560JXACBC" H 7050 3350 60  0001 C CNN "Mouse PN"
 	1    7050 3350
 	-1   0    0    -1
@@
 $EndComp
 $Comp
-L GND #PWR124
+L GND #PWR0129
 U 1 1 55A9AF9B
 P 7050 3500
-F 0 "#PWR124" H 7050 3250 50  0001 C CNN
+F 0 "#PWR0129" H 7050 3250 50  0001 C CNN
 F 1 "GND" H 7050 3350 50  0000 C CNN
 F 2 "" H 7050 3500 60  0000 C CNN
@@
 $EndComp
 $Comp
-L GND #PWR127
+L GND #PWR0130
 U 1 1 55A9B051
 P 7300 3500
-F 0 "#PWR127" H 7300 3250 50  0001 C CNN
+F 0 "#PWR0130" H 7300 3250 50  0001 C CNN
 F 1 "GND" H 7300 3350 50  0000 C CNN
 F 2 "" H 7300 3500 60  0000 C CNN
@@
 $EndComp
 $Comp
-L GND #PWR129
+L GND #PWR0131
 U 1 1 55A9FAF5
 P 9300 3600
-F 0 "#PWR129" H 9300 3350 50  0001 C CNN
+F 0 "#PWR0131" H 9300 3350 50  0001 C CNN
 F 1 "GND" H 9300 3450 50  0000 C CNN
 F 2 "" H 9300 3600 60  0000 C CNN
@@
 F 1 "SIM5320" H 3400 3150 60  0000 C CNN
 F 2 "CustomParts:SIM5320" H 2800 3650 60  0001 C CNN
-F 3 "http://www.simcom.ee/modules/wcdma-hspa/sim5320/" H 2800 3650 60  0001 C CNN
-F 4 "#" H 4150 2850 60  0001 C CNN "Mouse PN"
-F 5 "SIM5320A" H 4150 2850 60  0001 C CNN "AliExpress PN"
+F 3 "https://www.aliexpress.com/item/Original-SMT-type-WCDMA-module-SIM5320A/477453149.html" H 2800 3650 60  0001 C CNN
+F 4 "AliExpressOrder" H 4150 2850 60  0001 C CNN "Mouse PN"
 	1    4150 2850
 	1    0    0    -1
@@
 $EndComp
 $Comp
-L GND #PWR125
+L GND #PWR0132
 U 1 1 56099B91
 P 7150 1300
-F 0 "#PWR125" H 7150 1050 50  0001 C CNN
+F 0 "#PWR0132" H 7150 1050 50  0001 C CNN
 F 1 "GND" H 7150 1150 50  0000 C CNN
 F 2 "" H 7150 1300 60  0000 C CNN
